File: microSRCP/EAGLE/microSRCP/microSRCPProMiniV3.brd (EAGLE design)
At the start: 97.8 x 60.3 mm, 41 parts

Commit message: Detailkorrekturen
Connections:
- removed net S$31: DI0.5, DI2.5, DI3.5, DI4.5, DI6.5
- net 2-GND: now also E$4.4, E$4.6, E$5.4, E$5.6
- net GND: no longer E$4.4, E$4.6, E$5.4, E$5.6
- net S$29: now also DI0.5, DI2.5, DI3.5, DI4.5, DI6.5, DI7.5
Routing:
- net S$29: track 87.0 -> 102.2 mm
- net GND: track 198.2 -> 186.8 mm
- net 2-GND: track 129.5 -> 139.7 mm
- net S$31: track 10.2 -> 0.00 mm
- net S$6: track 101.7 -> 97.9 mm
- net 2-5V: track 131.3 -> 128.3 mm
- net S$5: track 89.8 -> 88.6 mm
Other:
- board text added: "+ +"
- board text added: "D C B A GND"
- board text added: "https://github.com/mc-b/microSRCP"
Changed lines of the file:
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@@
 <wire x1="97.79" y1="60.325" x2="0" y2="60.325" width="0.4064" layer="20"/>
 <wire x1="0" y1="60.325" x2="0" y2="0" width="0.4064" layer="20"/>
+<text x="38.735" y="20.32" size="1.27" layer="25">+    +</text>
+<text x="34.925" y="36.195" size="1.27" layer="25" distance="100">D
+C
+B
+A
+GND</text>
+<text x="14.605" y="53.975" size="1.778" layer="25">https://github.com/mc-b/microSRCP</text>
 </plain>
 <attributes>
@@
 <contactref element="GND" pad="2"/>
 <wire x1="55.88" y1="46.99" x2="49.53" y2="46.99" width="0.4064" layer="16"/>
+<contactref element="E$5" pad="6"/>
+<wire x1="81.915" y1="43.18" x2="84.455" y2="43.18" width="0.4064" layer="1"/>
+<contactref element="E$5" pad="4"/>
+<wire x1="84.455" y1="43.18" x2="86.995" y2="43.18" width="0.4064" layer="1"/>
+<contactref element="E$4" pad="6"/>
+<wire x1="90.805" y1="17.78" x2="88.265" y2="17.78" width="0.4064" layer="1"/>
+<contactref element="E$4" pad="4"/>
+<wire x1="88.265" y1="17.78" x2="85.725" y2="17.78" width="0.4064" layer="1"/>
 </signal>
 <signal name="2-5V">
@@
 <wire x1="93.98" y1="48.26" x2="83.185" y2="48.26" width="0.4064" layer="1"/>
 <wire x1="78.74" y1="45.72" x2="78.74" y2="44.45" width="0.4064" layer="1"/>
-<wire x1="73.66" y1="44.45" x2="73.66" y2="45.72" width="0.254" layer="1"/>
-<wire x1="72.39" y1="43.18" x2="73.66" y2="44.45" width="0.254" layer="1"/>
 <contactref element="D2" pad="2"/>
-<wire x1="71.12" y1="44.45" x2="73.66" y2="44.45" width="0.254" layer="16"/>
-<contactref element="D3~" pad="2"/>
-<contactref element="D4" pad="2"/>
-<wire x1="68.58" y1="44.45" x2="71.12" y2="44.45" width="0.254" layer="1"/>
-<contactref element="D5~" pad="2"/>
-<wire x1="66.04" y1="44.45" x2="68.58" y2="44.45" width="0.254" layer="1"/>
-<contactref element="D6~" pad="2"/>
-<wire x1="63.5" y1="44.45" x2="66.04" y2="44.45" width="0.254" layer="1"/>
-<contactref element="D7" pad="2"/>
-<wire x1="60.96" y1="44.45" x2="63.5" y2="44.45" width="0.254" layer="1"/>
-<contactref element="D8" pad="2"/>
-<wire x1="58.42" y1="44.45" x2="60.96" y2="44.45" width="0.254" layer="1"/>
-<contactref element="D9~" pad="2"/>
-<wire x1="58.42" y1="44.45" x2="55.88" y2="44.45" width="0.254" layer="1"/>
 <wire x1="78.74" y1="44.45" x2="73.66" y2="44.45" width="0.4064" layer="1"/>
 <contactref element="E$5" pad="7"/>
@@
 <contactref element="A6" pad="2"/>
 <wire x1="53.34" y1="16.51" x2="50.8" y2="16.51" width="0.4064" layer="16"/>
+<contactref element="D3~" pad="2"/>
+<contactref element="D4" pad="2"/>
+<wire x1="68.58" y1="44.45" x2="71.12" y2="44.45" width="0.4064" layer="1"/>
+<contactref element="D5~" pad="2"/>
+<wire x1="66.04" y1="44.45" x2="68.58" y2="44.45" width="0.4064" layer="1"/>
+<contactref element="D6~" pad="2"/>
+<wire x1="63.5" y1="44.45" x2="66.04" y2="44.45" width="0.4064" layer="1"/>
+<contactref element="D7" pad="2"/>
+<wire x1="60.96" y1="44.45" x2="63.5" y2="44.45" width="0.4064" layer="1"/>
+<contactref element="D8" pad="2"/>
+<wire x1="58.42" y1="44.45" x2="60.96" y2="44.45" width="0.4064" layer="1"/>
+<wire x1="58.42" y1="44.45" x2="55.88" y2="44.45" width="0.4064" layer="1"/>
+<contactref element="D9~" pad="2"/>
 <contactref element="GND" pad="1"/>
 <wire x1="55.88" y1="44.45" x2="49.53" y2="44.45" width="0.4064" layer="16"/>
+<wire x1="73.66" y1="44.45" x2="71.12" y2="44.45" width="0.4064" layer="1"/>
 </signal>
 <signal name="S$2">
@@
 <contactref element="D5~" pad="1"/>
 <wire x1="66.04" y1="38.1" x2="66.04" y2="41.91" width="0.4064" layer="16"/>
-<wire x1="66.04" y1="41.91" x2="64.77" y2="39.37" width="0.254" layer="1"/>
-<wire x1="64.77" y1="39.37" x2="52.07" y2="39.37" width="0.254" layer="1"/>
-<wire x1="52.07" y1="39.37" x2="52.07" y2="48.895" width="0.254" layer="1"/>
+<wire x1="66.04" y1="41.91" x2="64.77" y2="40.005" width="0.254" layer="1"/>
+<wire x1="64.77" y1="40.005" x2="52.07" y2="40.005" width="0.254" layer="1"/>
+<wire x1="52.07" y1="40.005" x2="52.07" y2="48.895" width="0.254" layer="1"/>
 <wire x1="52.07" y1="48.895" x2="9.525" y2="48.895" width="0.254" layer="1"/>
 <contactref element="MAX7219" pad="12"/>
@@
 <contactref element="D6~" pad="1"/>
 <wire x1="63.5" y1="38.1" x2="63.5" y2="41.91" width="0.4064" layer="16"/>
-<wire x1="63.5" y1="41.91" x2="62.865" y2="40.005" width="0.254" layer="1"/>
-<wire x1="62.865" y1="40.005" x2="53.34" y2="40.005" width="0.254" layer="1"/>
-<wire x1="53.34" y1="40.005" x2="53.34" y2="50.165" width="0.254" layer="1"/>
+<wire x1="63.5" y1="41.91" x2="62.865" y2="43.18" width="0.254" layer="1"/>
+<wire x1="62.865" y1="43.18" x2="53.34" y2="43.18" width="0.254" layer="1"/>
+<wire x1="53.34" y1="43.18" x2="53.34" y2="50.165" width="0.254" layer="1"/>
 <wire x1="53.34" y1="50.165" x2="6.985" y2="50.165" width="0.254" layer="1"/>
 <wire x1="6.985" y1="50.165" x2="6.985" y2="22.86" width="0.254" layer="1"/>
@@
 <wire x1="76.2" y1="34.29" x2="80.01" y2="34.29" width="0.4064" layer="1"/>
 <wire x1="92.71" y1="40.64" x2="92.71" y2="16.51" width="0.4064" layer="1"/>
-<wire x1="92.71" y1="16.51" x2="88.265" y2="16.51" width="0.4064" layer="1"/>
+<wire x1="92.71" y1="16.51" x2="81.915" y2="16.51" width="0.4064" layer="1"/>
 <contactref element="E$4" pad="1"/>
-<wire x1="88.265" y1="16.51" x2="85.725" y2="16.51" width="0.4064" layer="1"/>
-<wire x1="85.725" y1="16.51" x2="81.915" y2="16.51" width="0.4064" layer="1"/>
 <wire x1="81.915" y1="16.51" x2="81.915" y2="15.24" width="0.4064" layer="1"/>
-<contactref element="E$4" pad="4"/>
-<wire x1="85.725" y1="16.51" x2="85.725" y2="17.78" width="0.4064" layer="1"/>
-<contactref element="E$4" pad="6"/>
-<wire x1="88.265" y1="16.51" x2="88.265" y2="17.78" width="0.4064" layer="1"/>
 <contactref element="E$5" pad="1"/>
-<contactref element="E$5" pad="4"/>
-<wire x1="90.805" y1="44.45" x2="90.805" y2="45.72" width="0.4064" layer="1"/>
-<wire x1="90.805" y1="44.45" x2="86.995" y2="44.45" width="0.4064" layer="1"/>
-<wire x1="86.995" y1="44.45" x2="86.995" y2="43.18" width="0.4064" layer="1"/>
-<wire x1="86.995" y1="44.45" x2="84.455" y2="44.45" width="0.4064" layer="1"/>
-<contactref element="E$5" pad="6"/>
-<wire x1="84.455" y1="44.45" x2="84.455" y2="43.18" width="0.4064" layer="1"/>
-<wire x1="90.805" y1="44.45" x2="90.805" y2="40.64" width="0.4064" layer="1"/>
+<wire x1="90.805" y1="45.72" x2="90.805" y2="40.64" width="0.4064" layer="1"/>
 <wire x1="76.2" y1="36.195" x2="52.705" y2="36.195" width="0.4064" layer="1"/>
 <contactref element="I2C" pad="4"/>
@@
 <wire x1="27.305" y1="15.875" x2="27.305" y2="22.86" width="0.4064" layer="16"/>
 </signal>
-<signal name="S$31">
+<signal name="S$29">
+<contactref element="MAX7219" pad="23"/>
+<wire x1="34.925" y1="22.86" x2="34.925" y2="14.605" width="0.4064" layer="16"/>
+<wire x1="34.925" y1="14.605" x2="3.175" y2="14.605" width="0.4064" layer="16"/>
+<wire x1="3.175" y1="14.605" x2="3.175" y2="46.99" width="0.4064" layer="16"/>
+<contactref element="DI1" pad="5"/>
+<wire x1="3.175" y1="46.99" x2="15.24" y2="46.99" width="0.4064" layer="16"/>
+<contactref element="DI5" pad="5"/>
+<wire x1="15.24" y1="46.99" x2="17.78" y2="46.99" width="0.4064" layer="16"/>
+<contactref element="DI7" pad="5"/>
+<wire x1="17.78" y1="46.99" x2="20.32" y2="46.99" width="0.4064" layer="16"/>
 <contactref element="DI0" pad="5"/>
 <contactref element="DI4" pad="5"/>
@@
 <contactref element="DI3" pad="5"/>
 <wire x1="22.86" y1="46.99" x2="25.4" y2="46.99" width="0.4064" layer="16"/>
-</signal>
-<signal name="S$29">
-<contactref element="MAX7219" pad="23"/>
-<wire x1="34.925" y1="22.86" x2="34.925" y2="14.605" width="0.4064" layer="16"/>
-<wire x1="34.925" y1="14.605" x2="3.175" y2="14.605" width="0.4064" layer="16"/>
-<wire x1="3.175" y1="14.605" x2="3.175" y2="46.99" width="0.4064" layer="16"/>
-<contactref element="DI1" pad="5"/>
-<wire x1="3.175" y1="46.99" x2="15.24" y2="46.99" width="0.4064" layer="16"/>
-<contactref element="DI5" pad="5"/>
-<wire x1="15.24" y1="46.99" x2="17.78" y2="46.99" width="0.4064" layer="16"/>
+<wire x1="20.32" y1="46.99" x2="22.86" y2="46.99" width="0.4064" layer="16"/>
 </signal>
 <signal name="S$27">
